File: Lesson 4/EE-Workshop.sch (EAGLE design)
At the start: 1 part

Commit message: ee piano project
electrical engineering piano project
Parts:
- added C1, C2: 0.1uF, rcl:C-USC0805
- added IC1: NE555D, linear:NE555D
- added Q1: BCW66, transistor:BCW60-NPN-SOT23-BEC
- added R1: 3k, rcl:R-US_R0805
- added R10: 910, rcl:R-US_R0805
- added R2: 6.2k, rcl:R-US_R0805
- added R3, R9: 1k, rcl:R-US_R0805
- added R4: 390, rcl:R-US_R0805
- added R5: 1.5k, rcl:R-US_R0805
- added R6: 1.3k, rcl:R-US_R0805
- added R7: 620, rcl:R-US_R0805
- added R8: 1.1k, rcl:R-US_R0805
- added S1, S2, S3, S4, S5, S6, S7, S8: MOMENTARY-SWITCH-SPST-SMD-6.2MM-TALL, SparkFun-Switches:MOMENTARY-SWITCH-SPST-SMD-6.2MM-TALL
- added SG1: F/HMB, buzzer:F/HMB
- BATT: value AB3V -> AB9V
Connections:
- new net N$1: R10.1, R10.2, R9.2
Other:
- moved on the sheet: BATT
